File: nRF52810_HW/nRF52810.kicad_pcb (KiCad board)
At the start: 2 copper layers, 39.8 x 31.4 mm, 32 parts, among them J1 TC2050-IDC-NL, SW1 TS-1088-AR02016, U1 AP2114HA-3.3TRG1, U2 NRF52810-QCAA-R, X1 SC-20S32.768kHz20PPM9pF, X2 XL7EL89CKI-111YLC-32M

Commit message: Considerate changes
Connections:
- U2 pad 19: unconnected-(U2-ANT-Pad19) -> (no net)

Commit message: bump large
Parts:
- removed LED1, LED2: LTST-C190KRKT, my_lib:[LED]Lite-On LTST-C190KRKT
- removed SW1: TS-1088-AR02016, my_lib:[TACTILE_SWITCH]XUNPU TS-1088-AR02016
- added ANT1: DN007, pepy_sym_lib:[ANTENNA]DN007_1,2.4GHz, F.Cu at (92.7, 119.2)
- added C15: CC0805KRX7R9BB104, pepy_sym_lib:[CAP_SMD_0805_2012Metric], F.Cu at (77.7, 135.6)
- added C16: CL21A106KOQNNNE, pepy_sym_lib:[CAP_SMD_0805_2012Metric], F.Cu at (63.1, 151.4)
- added C17: CL21A106KOQNNNE, pepy_sym_lib:[CAP_SMD_0805_2012Metric], F.Cu at (67.7, 151.4)
- added C18: CL21A106KOQNNNE, pepy_sym_lib:[CAP_SMD_0805_2012Metric], F.Cu at (74.6, 146.1)
- added C19: CL21A106KOQNNNE, pepy_sym_lib:[CAP_SMD_0805_2012Metric], F.Cu at (74.6, 141.1)
- added C20: C0805C105M4VACTU, pepy_sym_lib:[CAP_SMD_0805_2012Metric], F.Cu at (52.0, 116.1)
- added C21: C0805C105M4VACTU, pepy_sym_lib:[CAP_SMD_0805_2012Metric], F.Cu at (57.3, 115.3)
- added C22: CC0805KRX7R9BB104, pepy_sym_lib:[CAP_SMD_0805_2012Metric], F.Cu at (78.5, 128.4)
- added C23: CC0805KRX7R9BB104, pepy_sym_lib:[CAP_SMD_0805_2012Metric], F.Cu at (78.3, 130.8)
- added D2: LTST-C190KRKT, pepy_sym_lib:[LED]Lite-On LTST-C190KRKT, F.Cu at (83.5, 127.1)
- added H4: X6511WV-02H-C30D60, pepy_sym_lib:[2x1_PIN_HEADER_STR]XKB Connection X6511WV-02H-C60D30, F.Cu at (60.3, 146.9)
- added H5: X6511WV-02H-C30D60, pepy_sym_lib:[2x1_PIN_HEADER_STR]XKB Connection X6511WV-02H-C60D30, F.Cu at (62.4, 131.5)
- added H6: X6511WV-02H-C30D60, pepy_sym_lib:[2x1_PIN_HEADER_STR]XKB Connection X6511WV-02H-C60D30, F.Cu at (59.6, 131.5)
- added L1: LQG15HS1N0S02D, pepy_sym_lib:[IND_SMD_0402_1005Metric], F.Cu at (78.2, 117.3)
- added L2: FNR3015S4R7MT, pepy_sym_lib:[POWER_IND]cjiang (Changjiang Microelectronics Tech) FNR3015S4R7MT, F.Cu at (71.2, 144.7)
- added MH1: ~, pepy_sym_lib:[MOUNTING_HOLE]MountingHole_2.2mm_M2_DIN965_Pad, F.Cu at (44.6, 153.8)
- added MH2: ~, pepy_sym_lib:[MOUNTING_HOLE]MountingHole_2.2mm_M2_DIN965_Pad, F.Cu at (82.8, 153.5)
- added MH3: ~, pepy_sym_lib:[MOUNTING_HOLE]MountingHole_2.2mm_M2_DIN965_Pad, F.Cu at (48.7, 103.5)
- added MH4: ~, pepy_sym_lib:[MOUNTING_HOLE]MountingHole_2.2mm_M2_DIN965_Pad, F.Cu at (81.9, 104.1)
- added Q1: BSS138PW,115, pepy_sym_lib:[NMOS]Nexperia BSS138PW,115, F.Cu at (83.9, 124.1)
- added R10: 0805W8F1002T5E, pepy_sym_lib:[RES_SMD_0805_2012Metric], F.Cu at (52.0, 119.8)
- added R11: 0805W8F1002T5E, pepy_sym_lib:[RES_SMD_0805_2012Metric], F.Cu at (57.3, 118.9)
- added R12: 0805W8F1004T5E, pepy_sym_lib:[RES_SMD_0805_2012Metric], F.Cu at (79.9, 141.6)
- added R13: 0805W8F0000T5E, pepy_sym_lib:[RES_SMD_0805_2012Metric], F.Cu at (78.4, 124.2)
- added R14: RK73H2ATTD3573F, pepy_sym_lib:[RES_SMD_0805_2012Metric], F.Cu at (77.9, 141.6)
- added R15: 0805W8F0000T5E, pepy_sym_lib:[RES_SMD_0805_2012Metric], F.Cu at (78.3, 126.2)
- added R4: 0402WGF0000TCE, pepy_sym_lib:[RES_SMD_0402_1005Metric], F.Cu at (84.2, 117.2)
- added R5: 0402WGF0000TCE, pepy_sym_lib:[RES_SMD_0402_1005Metric], F.Cu at (74.8, 117.8)
- added R6: 0402WGF0000TCE, pepy_sym_lib:[RES_SMD_0402_1005Metric], F.Cu at (84.7, 116.8)
- added R7: 0805W8F4700T5E, pepy_sym_lib:[RES_SMD_0805_2012Metric], F.Cu at (84.8, 120.9)
- added R8: 0805W8F1000T5E, pepy_sym_lib:[RES_SMD_0805_2012Metric], F.Cu at (72.7, 139.1)
- added RF1: U.FL-R-SMT-1(80), pepy_sym_lib:[SMD_COAXIAL_CONNECTOR]HRS(Hirose) U.FL-R-SMT-1(80), F.Cu at (84.7, 114.3)
- added RF2: U.FL-R-SMT-1(80), pepy_sym_lib:[SMD_COAXIAL_CONNECTOR]HRS(Hirose) U.FL-R-SMT-1(80), F.Cu at (78.6, 119.9)
- added S1: TS-1088-AR02016, pepy_sym_lib:[TACTILE_SWITCH]XUNPU TS-1088-AR02016, F.Cu at (49.3, 119.4)
- added S2: TS-1088-AR02016, pepy_sym_lib:[TACTILE_SWITCH]XUNPU TS-1088-AR02016, F.Cu at (54.7, 119.3)
- added TP1: VBAT, pepy_sym_lib:[TEST_POINT]TestPoint_Pad_2.0x2.0mm, F.Cu at (50.5, 138.6)
- added TP2: GND, pepy_sym_lib:[TEST_POINT]TestPoint_Pad_2.0x2.0mm, F.Cu at (50.4, 142.0)
- added U3: AP2114HA-3.3TRG1, pepy_sym_lib:[LDO]Diodes Incorporated AP2114HA-3.3TRG1, F.Cu at (65.4, 145.0)
- added U4: TPS61220DCKR, pepy_sym_lib:[BOOST_CONV]Texas Instruments TPS61220DCKR, F.Cu at (74.5, 143.3)
- added X3: WJ500V-5.08-2P-14-00A, pepy_sym_lib:[1x2_SCREW_TERMINAL_BLOCK]Ningbo Kangnex Elec WJ500V-5.08-2P, F.Cu at (52.9, 150.5)
- C1, C2: value 22u -> C0805C100K5GACTU; footprint Capacitor_SMD:C_0805_2012Metric -> pepy_sym_lib:[CAP_SMD_0805_2012Metric]
- C10, C5: value 100nF -> CC0805KRX7R9BB104; footprint Capacitor_SMD:C_0805_2012Metric -> pepy_sym_lib:[CAP_SMD_0805_2012Metric]
- C11: value 100pF -> CC0805KRX7R9BB104; footprint Capacitor_SMD:C_0805_2012Metric -> pepy_sym_lib:[CAP_SMD_0805_2012Metric]
- C12: value 12pF -> CC0805KRX7R9BB104; footprint Capacitor_SMD:C_0805_2012Metric -> pepy_sym_lib:[CAP_SMD_0805_2012Metric]
- C13: value 12pF -> C0805C101K5GACTU; footprint Capacitor_SMD:C_0805_2012Metric -> pepy_sym_lib:[CAP_SMD_0805_2012Metric]
- C14: value 1u -> CL21A475KAQNNNE; footprint Capacitor_SMD:C_0805_2012Metric -> pepy_sym_lib:[CAP_SMD_0805_2012Metric]
- C3, C4: value 12pF -> C0805C120J5GACAUTO; footprint Capacitor_SMD:C_0805_2012Metric -> pepy_sym_lib:[CAP_SMD_0805_2012Metric]
- C6: value 100nF -> CL21A475KAQNNNE; footprint Capacitor_SMD:C_0805_2012Metric -> pepy_sym_lib:[CAP_SMD_0805_2012Metric]
- C7: value 1uF -> C0805C105M4VACTU; footprint Capacitor_SMD:C_0805_2012Metric -> pepy_sym_lib:[CAP_SMD_0805_2012Metric]
- C8: value 100pF -> C0805C120J5GACAUTO; footprint Capacitor_SMD:C_0805_2012Metric -> pepy_sym_lib:[CAP_SMD_0805_2012Metric]
- C9: value 4.7u -> C0805C120J5GACAUTO; footprint Capacitor_SMD:C_0805_2012Metric -> pepy_sym_lib:[CAP_SMD_0805_2012Metric]
- D1: value STPS140Z -> LTST-C190KRKT; footprint my_lib:SOD-123_L2.8-W1.8-LS3.7-RD -> pepy_sym_lib:[LED]Lite-On LTST-C190KRKT
- H1, H2, H3: value MountingHole_Pad -> X6511WV-02H-C30D60; footprint MountingHole:MountingHole_2.2mm_M2_DIN965_Pad -> pepy_sym_lib:[2x1_PIN_HEADER_STR]XKB Connection X6511WV-02H-C60D30
- J1: footprint my_lib:[PLUG_OF_NAILS_10P]TC2050_IDC_NL -> pepy_sym_lib:[PLUG_OF_NAILS_10P]TC2050_IDC_NL
- R1: value 470R -> 0805W8F4700T5E; footprint Resistor_SMD:R_0805_2012Metric -> pepy_sym_lib:[RES_SMD_0805_2012Metric]
- R2: value 470R -> 0402WGF0000TCE; footprint Resistor_SMD:R_0805_2012Metric -> pepy_sym_lib:[RES_SMD_0402_1005Metric]
- R3: value 10k -> 0402WGF0000TCE; footprint Resistor_SMD:R_0805_2012Metric -> pepy_sym_lib:[RES_SMD_0402_1005Metric]
- U1: value AP2114HA-3.3TRG1 -> NRF52810-QCAA-R; footprint my_lib:[LDO]Diodes Incorporated AP2114HA-3.3TRG1 -> pepy_sym_lib:[MCU]Nordic Semicon nRF52810-QCAA-R
- U2: value NRF52810-QCAA-R -> PMW3360DM-T2QU; footprint my_lib:[MCU]Nordic Semicon nRF52810-QCAA-R -> pepy_sym_lib:[OPTICAL_NAVIGATION_CHIP]PixArt PMW3360DM-T2QU
- X1: value SC-20S32.768kHz20PPM9pF -> XL7EL89CKI-111YLC-32M; footprint my_lib:[Crystal_32_768_kHZ]Seiko SC-20S,32.768kHz,20PPM,9pF -> pepy_sym_lib:[Crystal_32_MHz]YXC XL7EL89CKI-111YLC-32M
- X2: value XL7EL89CKI-111YLC-32M -> SC-20S32.768kHz20PPM9pF; footprint my_lib:[Crystal_32_MHz]YXC XL7EL89CKI-111YLC-32M -> pepy_sym_lib:[Crystal_32_768_kHZ]Seiko SC-20S,32.768kHz,20PPM,9pF
- moved D1 125.1 mm to (57.6, 156.7)
- moved H3 119.1 mm to (55.3, 142.9)
- moved H2 115.1 mm to (55.3, 140.3)
- moved R1 110.8 mm to (60.1, 155.8), turned to -90 degrees
- moved J1 105.4 mm to (52.1, 127.3)
- moved FID3 99.0 mm to (83.3, 139.1)
- moved C14 96.3 mm to (78.4, 132.8), turned to 0 degrees
- moved C9 94.6 mm to (62.4, 114.5), turned to 0 degrees
- moved C5 93.6 mm to (65.7, 109.9), turned to -90 degrees
- moved U2 92.3 mm to (70.3, 129.8), turned to 180 degrees
- moved C6 91.6 mm to (67.8, 111.3), turned to -90 degrees
- moved C3 91.0 mm to (72.7, 111.6), turned to -90 degrees
- moved H1 90.8 mm to (55.2, 137.6)
- moved C4 89.7 mm to (75.3, 114.6), turned to 180 degrees
- moved C8 88.9 mm to (62.4, 112.5), turned to 0 degrees
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Connections:
- C1 pad 1: /V_INPUT -> GND
- C1 pad 2: GND -> Net-(C1-Pad2)
- C10 pad 1: +3.3V -> GND
- C10 pad 2: GND -> /VDD_MCU
- C11 pad 1: +3.3V -> GND
- C11 pad 2: GND -> /VDD_MCU
- C12 pad 1: /XC1 -> GND
- C12 pad 2: GND -> Net-(U1-DEC2)
- C13 pad 1: /XC2 -> GND
- C13 pad 2: GND -> Net-(U1-DEC3)
- C14 pad 1: /BUTTON -> Net-(U2-VDDPIX)
- C2 pad 1: +3.3V -> GND
- C2 pad 2: GND -> Net-(C2-Pad2)
- C3 pad 1: Net-(U2-P0.00/XL1) -> GND
- C3 pad 2: GND -> /XC2
- C4 pad 1: Net-(U2-P0.01/XL2) -> GND
- C4 pad 2: GND -> /XC1
- C5 pad 1: Net-(U2-DEC1) -> GND
- C5 pad 2: GND -> Net-(U1-DEC1)
- C6 pad 1: +3.3V -> GND
- C6 pad 2: GND -> /VDD_MCU
- C7 pad 1: Net-(U2-DEC4) -> GND
- C7 pad 2: GND -> Net-(U1-DEC4)
- C8 pad 1: Net-(U2-DEC2) -> GND
- C8 pad 2: GND -> Net-(U1-P0.00/XL1)
- C9 pad 1: +3.3V -> GND
- C9 pad 2: GND -> Net-(U1-P0.01/XL2)
- D1 pad 1: /BUTTON -> Net-(D1-A)
- H1 pad 1: GND -> /VDBG
- H2 pad 1: GND -> /VBAT
- H3 pad 1: GND -> /VEXT
- J1 pad 1: +3.3V -> /VDD_MCU
- J1 pad 10: GND -> /nRESET
- J1 pad 2: unconnected-(J1-Pad2) -> /SWDIO
- J1 pad 3: /V_INPUT -> GND
- J1 pad 4: /nRESET -> /SWDCLK
- J1 pad 5: /SWDIO -> /GEN
- J1 pad 6: /SWDCLK -> unconnected-(J1-Pad6)
- J1 pad 7: unconnected-(J1-Pad7) -> /VDBG
- J1 pad 8: /GEN1 -> unconnected-(J1-Pad8)
- R1 pad 1: +3.3V -> /VIN
- R1 pad 2: Net-(LED1-A) -> Net-(D1-A)
- R2 pad 1: /P0.20 -> /ANT
- R2 pad 2: Net-(LED2-A) -> Net-(C1-Pad2)
- R3 pad 1: +3.3V -> Net-(L1-Pad1)
- R3 pad 2: /BUTTON -> Net-(C2-Pad2)
- U1 pad 1: /V_INPUT -> Net-(U1-DEC1)
- U1 pad 2: GND -> Net-(U1-P0.00/XL1)
- U1 pad 3: +3.3V -> Net-(U1-P0.01/XL2)
- U1 pad 4: GND -> unconnected-(U1-P0.04/AIN2-Pad4)
- U2 pad 1: Net-(U2-DEC1) -> unconnected-(U2-NC-Pad1)
- U2 pad 10: unconnected-(U2-P0.12-Pad10) -> /SCLK
- U2 pad 11: unconnected-(U2-P0.14-Pad11) -> /MOSI
- U2 pad 12: unconnected-(U2-P0.15-Pad12) -> /MISO
- U2 pad 13: /BUTTON -> /nCS
- U2 pad 14: /GEN1 -> unconnected-(U2-NC-Pad14)
- U2 pad 15: /P0.20 -> Net-(U2-LED_P)
- U2 pad 16: /nRESET -> unconnected-(U2-NC-Pad16)
- U2 pad 2: Net-(U2-P0.00/XL1) -> unconnected-(U2-NC-Pad2)
- U2 pad 3: Net-(U2-P0.01/XL2) -> Net-(U2-VDDPIX)
- U2 pad 4: unconnected-(U2-P0.04/AIN2-Pad4) -> /VDD_1.9V
- U2 pad 5: unconnected-(U2-P0.05/AIN3-Pad5) -> /VDD_MCU
- U2 pad 7: unconnected-(U2-P0.09-Pad7) -> /nRST_PMW
- U2 pad 8: unconnected-(U2-P0.10-Pad8) -> GND
- U2 pad 9: +3.3V -> /MTN_INT
- X1 pad 1: Net-(U2-P0.01/XL2) -> /XC1
- X1 pad 2: Net-(U2-P0.00/XL1) -> GND
- X2 pad 1: /XC1 -> Net-(U1-P0.00/XL1)
- X2 pad 2: GND -> Net-(U1-P0.01/XL2)
Routing:
- net +3.3V: track 94.7 -> 0.00 mm, vias 2 -> 0
- net /VDD_MCU: track 0.00 -> 74.0 mm, vias 0 -> 5
- net /VIN: track 0.00 -> 54.1 mm
- net /GEN: track 0.00 -> 34.5 mm, vias 0 -> 2
- net /VDD_1.9V: track 0.00 -> 33.6 mm
- net GND: track 34.4 -> 67.2 mm, vias 42 -> 43
- net /LEFT: track 0.00 -> 27.2 mm
- net /nRST_MAN: track 0.00 -> 24.0 mm, vias 0 -> 2
- net /BUTTON: track 23.0 -> 0.00 mm
- net /nRESET: track 12.9 -> 33.2 mm
- net /SWDCLK: track 12.9 -> 33.0 mm, vias 0 -> 2
- net /nCS: track 0.00 -> 18.5 mm
- net /SWDIO: track 13.0 -> 30.4 mm, vias 0 -> 2
- net /MISO: track 0.00 -> 16.6 mm
- net /RIGHT: track 0.00 -> 15.0 mm
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- added copper zone on F.Cu, net /VDD_1.9V
- added copper zone on F.Cu, net /VDD_3.3V
- added copper zone on B.Cu, net /VDD_MCU
- added copper zone on F.Cu, net /VDD_MCU
- added copper zone on F.Cu, net /VIN
- added copper zone on In1.Cu, net GND
- added copper zone on In2.Cu, net GND
- removed copper zone on B.Cu, net GND
Other:
- board size 39.8 x 31.4 mm -> 62.2 x 65.2 mm
- copper layers 2 -> 4
- board text added: "0"
- board text added: "0 mm"
- board text added: "0.01 mm"
- board text added: "0.0152 mm"
- board text added: "0.02"
- board text added: "0.035 mm"
- board text added: "0.0994 mm"
- board text added: "1"
- board text added: "1.265 mm"
- board text added: "3.3"
- board text added: "4.5"
- board text added: "B.Cu"
- board text added: "B.Mask"
- board text added: "B.Paste"
- board text added: "B.Silkscreen"
- board text added: "Bottom Silk Screen"
- board text added: "Bottom Solder Mask"
- board text added: "Bottom Solder Paste"
- board text added: "Color"
- board text added: "Dielectric 1"
- board text added: "Dielectric 2"
- board text added: "Dielectric 3"
- board text added: "Epsilon R"
- board text added: "F.Cu"
- board text added: "F.Mask"
- board text added: "F.Paste"
- board text added: "F.Silkscreen"
- board text added: "FR4"
- board text added: "In1.Cu"
- board text added: "In2.Cu"
- board text added: "Layer Name"
- board text added: "Loss Tangent"
- board text added: "Material"
- board text added: "Not specified"
- board text added: "Thickness (mm)"
- board text added: "Top Silk Screen"
- board text added: "Top Solder Mask"
- board text added: "Top Solder Paste"
- board text added: "Type"
- board text added: "copper"
- board text added: "core"
- board text added: "prepreg"
- board text removed: "Project: nRF52810 v1 Designed by: perseluspy"

Commit message: Bulk change
Parts:
- moved D2 40.2 mm to (45.5, 114.0), turned to 90 degrees
- moved R7 39.3 mm to (45.5, 120.1), turned to 90 degrees
- moved Q1 39.1 mm to (45.4, 116.9), turned to 0 degrees
- moved FID2 14.9 mm to (70.0, 101.0), turned to 180 degrees
- moved MH4 5.61 mm to (76.4, 103.2)
- moved FID3 5.28 mm to (87.2, 142.6)
- moved R1 4.56 mm to (57.5, 152.0)
- moved H6 3.89 mm to (56.7, 134.0)
- moved H5 3.83 mm to (59.5, 134.0)
- moved C16 3.77 mm to (60.4, 154.0)
- moved C17 3.77 mm to (65.0, 154.0)
- moved MH1 3.63 mm to (43.0, 157.1)
- moved U3 3.45 mm to (62.8, 147.3)
- moved ANT1 3.30 mm to (94.5, 116.4)
- moved TP2 3.24 mm to (47.2, 142.0)
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Connections:
- U1 pad 15: /LED -> /nRST_MAN
- U1 pad 7: /GEN -> /LED
- U1 pad 8: /nRST_MAN -> /GEN
Routing:
- net /VIN: track 54.1 -> 75.9 mm
- net /VDD_MCU: track 74.0 -> 83.8 mm, vias 5 -> 6
- net /nRST_MAN: track 24.0 -> 15.6 mm, vias 2 -> 0
- net /LED: track 14.4 -> 21.5 mm
- net /VDD_1.9V: track 33.6 -> 26.6 mm
- net GND: track 67.2 -> 73.7 mm, vias 43 -> 78
- net /nRESET: track 33.2 -> 27.2 mm
- net /SWDCLK: track 33.0 -> 37.7 mm
- net /SWDIO: track 30.4 -> 34.9 mm
- net /GEN: track 34.5 -> 38.0 mm
- net /VIN_LDO: track 5.39 -> 2.49 mm
- net /XC2: track 6.86 -> 4.47 mm
- net /nCS: track 18.5 -> 20.7 mm
- net /MISO: track 16.6 -> 18.7 mm
- net /MOSI: track 14.9 -> 16.9 mm
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- added copper zone on F.Cu, net /VIN_LDO
- added copper zone on F.Cu, net GND
Other:
- board size 62.2 x 65.2 mm -> 59 x 65.2 mm
- board text added: "4.1"

Commit message: test_phase
Parts:
- added TP3: Vtref, pepy_sym_lib:[TEST_POINT]TestPoint_Pad_D1.0mm, F.Cu at (58.1, 124.6)
- added TP4: LED, pepy_sym_lib:[TEST_POINT]TestPoint_Pad_D1.0mm, F.Cu at (47.5, 113.9)
- added TP5: LEFT, pepy_sym_lib:[TEST_POINT]TestPoint_Pad_D1.0mm, F.Cu at (49.5, 112.3)
- added TP6: RIGHT, pepy_sym_lib:[TEST_POINT]TestPoint_Pad_D1.0mm, F.Cu at (59.5, 118.8)
- added TP7: nRESET, pepy_sym_lib:[TEST_POINT]TestPoint_Pad_D1.0mm, F.Cu at (81.2, 125.0)
- moved MH2 4.24 mm to (80.0, 156.4)
- moved R15 2.44 mm to (77.1, 126.0)
- moved FID3 2.16 mm to (85.0, 142.8)
- moved FID1 2.16 mm to (48.2, 110.0)
- moved R13 1.55 mm to (77.0, 128.1)
- moved MH1 0.51 mm to (42.9, 157.6)
- moved FID2 0.39 mm to (69.8, 101.3)
- moved C4 0.09 mm to (74.7, 114.2)
Routing:
- net /nRESET: track 27.2 -> 40.4 mm
- net /nRST_PMW: track 4.36 -> 13.2 mm
- net GND: track 73.7 -> 79.2 mm, vias 78 -> 207
- net /nRST_MAN: track 15.6 -> 11.0 mm
- net /VDD_MCU: track 83.8 -> 87.8 mm
- net /LED: track 21.5 -> 25.3 mm
- net /RIGHT: track 15.0 -> 17.5 mm
- net /LEFT: track 27.2 -> 29.7 mm
- net /SWDIO: track 34.9 -> 36.5 mm
