File: nRF52810_HW/nRF52810.kicad_sch (KiCad schematic)
At the start: 32 parts, among them J1 TC2050-IDC-NL, SW1 TS-1088-AR02016, U1 AP2114HA-3.3TRG1, U2 NRF52810-QCAA-R, X1 SC-20S32.768kHz20PPM9pF, X2 XL7EL89CKI-111YLC-32M

Commit message: commit++
Parts:
- removed C1, C2: 22u, Capacitor_SMD:C_0805_2012Metric, symbol Device:C
- removed C10, C5, C6: 100nF, Capacitor_SMD:C_0805_2012Metric, symbol Device:C_Small
- removed C14: 1u, Capacitor_SMD:C_0805_2012Metric, symbol Device:C
- removed C7: 1uF, Capacitor_SMD:C_0805_2012Metric, symbol Device:C_Small
- removed D1: STPS140Z, my_lib:SOD-123_L2.8-W1.8-LS3.7-RD, symbol my_symbol_library:STPS140Z
- removed H1, H2, H3: MountingHole_Pad, MountingHole:MountingHole_2.2mm_M2_DIN965_Pad, symbol Mechanical:MountingHole_Pad
- removed J1: TC2050-IDC-NL, my_lib:[PLUG_OF_NAILS_10P]TC2050_IDC_NL, symbol my_symbol_library:TC2050-IDC-NL
- removed LED1, LED2: LTST-C190KRKT, my_lib:[LED]Lite-On LTST-C190KRKT, symbol my_symbol_library:LTST-C190KRKT
- removed R1, R2: 470R, Resistor_SMD:R_0805_2012Metric, symbol Device:R_Small
- removed R3: 10k, Resistor_SMD:R_0805_2012Metric, symbol Device:R
- removed SW1: TS-1088-AR02016, my_lib:[TACTILE_SWITCH]XUNPU TS-1088-AR02016, symbol my_symbol_library:TS-1088-AR02016
- removed U1: AP2114HA-3.3TRG1, my_lib:[LDO]Diodes Incorporated AP2114HA-3.3TRG1, symbol my_symbol_library:AP2114HA-3.3TRG1
- added C? (x2): CL21A106KOQNNNE, pepy_sym_lib:[CAP_SMD_0805_2012Metric], symbol pepy_sym_lib:[CAP_SMD_0805_2012Metric]Samsung Electro-Mechanics CL21A106KOQNNNE
- added C? (x3): CC0805KRX7R9BB104, pepy_sym_lib:[CAP_SMD_0805_2012Metric], symbol pepy_sym_lib:[CAP_SMD_0805_2012Metric]YAGEO CC0805KRX7R9BB104
- added C? (x2): C0805C105M4VACTU, pepy_sym_lib:[CAP_SMD_0805_2012Metric], symbol pepy_sym_lib:[CAP_SMD_0805_2012Metric]KEMET C0805C105M4VACTU
- added D?: STPS140Z, pepy_sym_lib:[SCHOTTKY_DIODE_40V]STMicroelectronics STPS140Z, symbol pepy_sym_lib:[SCHOTTKY_DIODE_40V]STMicroelectronics STPS140Z
- added D? (x2): LTST-C190KRKT, pepy_sym_lib:[LED]Lite-On LTST-C190KRKT, symbol pepy_sym_lib:[LED]Lite-On LTST-C190KRKT
- added J?: TC2050-IDC-NL, pepy_sym_lib:[PLUG_OF_NAILS_10P]TC2050_IDC_NL, symbol pepy_sym_lib:[PLUG_OF_NAILS_10P]TC2050_IDC_NL
- added MH? (x3): ~, pepy_sym_lib:[MOUNTING_HOLE]MountingHole_2.2mm_M2_DIN965_Pad, symbol pepy_sym_lib:[MOUNTING_HOLE]MountingHole_Pad
- added R? (x2): 0805W8F4700T5E, pepy_sym_lib:[RES_SMD_0805_2012Metric], symbol pepy_sym_lib:[RES_SMD_0805_2012Metric]UNI-ROYAL(Uniroyal Elec) 0805W8F4700T5E
- added R?: 0805W8F1002T5E, pepy_sym_lib:[RES_SMD_0805_2012Metric], symbol pepy_sym_lib:[RES_SMD_0805_2012Metric]UNI-ROYAL(Uniroyal Elec) 0805W8F1002T5E
- added S?: TS-1088-AR02016, pepy_sym_lib:[TACTILE_SWITCH]XUNPU TS-1088-AR02016, symbol pepy_sym_lib:[TACTILE_SWITCH]XUNPU TS-1088-AR02016
- added U?: AP2114HA-3.3TRG1, pepy_sym_lib:[LDO]Diodes Incorporated AP2114HA-3.3TRG1, symbol pepy_sym_lib:[LDO]Diodes Incorporated AP2114HA-3.3TRG1
Connections:
- net +3.3V: now also C?.2, C?.2, C?.2, J?.1, R?.1, R?.2, U?.3 (OUT)
- net BUTTON: now also C?.2, D?.1 (C), R?.1, S?.2
- net GND: now also C?.1, C?.1, C?.1, C?.1, C?.1, C?.1, C?.1, D?.2 (A), D?.2 (C), D?.2 (C), J?.3, J?.5, MH?.1, MH?.1, MH?.1, S?.1, U?.2 (GND), U?.4 (GND)
- net P0.20: now also R?.1
- net SWDCLK: now also J?.4
- net SWDIO: now also J?.2
- net V_INPUT: now also C?.2, J?.7, U?.1 (IN)
- net nRESET: now also J?.10
- net at U2.30 (DEC4): now also C?.2
- net at U2.1 (DEC1): now also C?.2
- new net: D?.1 (A), R?.2 (x2)

Commit message: Latest
Parts:
- removed C12, C13, C3, C4: 12pF, Capacitor_SMD:C_0805_2012Metric, symbol Device:C_Small
- added C? (x4): C0805C120J5GACAUTO, pepy_sym_lib:[CAP_SMD_0805_2012Metric], symbol pepy_sym_lib:[CAP_SMD_0805_2012Metric]KEMET C0805C120J5GACAUTO
Connections:
- net GND: now also C?.1, C?.1, C?.1, C?.2
- net XC1: now also C?.2
- net XC2: now also C?.2
- net at U2.2 (P0.00/XL1), X1.2: now also C?.1
- net at U2.3 (P0.01/XL2), X1.1: now also C?.2

Commit message: Considerate changes
Parts:
- removed C? (x2): CL21A106KOQNNNE, pepy_sym_lib:[CAP_SMD_0805_2012Metric], symbol pepy_sym_lib:[CAP_SMD_0805_2012Metric]Samsung Electro-Mechanics CL21A106KOQNNNE
- removed C?: C0805C105M4VACTU, pepy_sym_lib:[CAP_SMD_0805_2012Metric], symbol pepy_sym_lib:[CAP_SMD_0805_2012Metric]KEMET C0805C105M4VACTU
- removed D?: STPS140Z, pepy_sym_lib:[SCHOTTKY_DIODE_40V]STMicroelectronics STPS140Z, symbol pepy_sym_lib:[SCHOTTKY_DIODE_40V]STMicroelectronics STPS140Z
- removed R?: 0805W8F1002T5E, pepy_sym_lib:[RES_SMD_0805_2012Metric], symbol pepy_sym_lib:[RES_SMD_0805_2012Metric]UNI-ROYAL(Uniroyal Elec) 0805W8F1002T5E
- removed S?: TS-1088-AR02016, pepy_sym_lib:[TACTILE_SWITCH]XUNPU TS-1088-AR02016, symbol pepy_sym_lib:[TACTILE_SWITCH]XUNPU TS-1088-AR02016
- removed U?: AP2114HA-3.3TRG1, pepy_sym_lib:[LDO]Diodes Incorporated AP2114HA-3.3TRG1, symbol pepy_sym_lib:[LDO]Diodes Incorporated AP2114HA-3.3TRG1
- added ANT2: DN007, pepy_sym_lib:[ANTENNA]DN007_1,2.4GHz, symbol pepy_sym_lib:[ANTENNA]DN007*1,2.4GHz
- added C1, C17, C2, C20: CL21A106KOQNNNE, pepy_sym_lib:[CAP_SMD_0805_2012Metric], symbol pepy_sym_lib:[CAP_SMD_0805_2012Metric]Samsung Electro-Mechanics CL21A106KOQNNNE
- added C15, C16: C0805C100K5GACTU, pepy_sym_lib:[CAP_SMD_0805_2012Metric], symbol pepy_sym_lib:[CAP_SMD_0805_2012Metric]KEMET C0805C100K5GACTU
- added C18: CC0805KRX7R9BB104, pepy_sym_lib:[CAP_SMD_0805_2012Metric], symbol pepy_sym_lib:[CAP_SMD_0805_2012Metric]YAGEO CC0805KRX7R9BB104
- added C19: CL21A475KAQNNNE, pepy_sym_lib:[CAP_SMD_0805_2012Metric], symbol pepy_sym_lib:[CAP_SMD_0805_2012Metric]Samsung Electro-Mechanics CL21A475KAQNNNE
- added C3: C0805C105M4VACTU, pepy_sym_lib:[CAP_SMD_0805_2012Metric], symbol pepy_sym_lib:[CAP_SMD_0805_2012Metric]KEMET C0805C105M4VACTU
- added H1, H2, H3, H4, H5, H6: X6511WV-02H-C30D60, pepy_sym_lib:[2x1_PIN_HEADER_STR]XKB Connection X6511WV-02H-C60D30, symbol pepy_sym_lib:[2x1_PIN_HEADER_STR]XKB Connection X6511WV-02H-C60D30
- added L1: LQG15HS1N0S02D, pepy_sym_lib:[IND_SMD_0402_1005Metric], symbol pepy_sym_lib:[IND_SMD_0402_1005Metric]Murata Electronics LQG15HS1N0S02D
- added L2: FNR3015S4R7MT, pepy_sym_lib:[POWER_IND]cjiang (Changjiang Microelectronics Tech) FNR3015S4R7MT, symbol pepy_sym_lib:[POWER_IND]cjiang (Changjiang Microelectronics Tech) FNR3015S4R7MT
- added Q1: BSS138PW,115, pepy_sym_lib:[NMOS]Nexperia BSS138PW,115, symbol pepy_sym_lib:[NMOS]Nexperia BSS138PW,115
- added R10, R6, R7, R8, R9: 0402WGF0000TCE, pepy_sym_lib:[RES_SMD_0402_1005Metric], symbol pepy_sym_lib:[RES_SMD_0402_1005Metric]UNI-ROYAL(Uniroyal Elec) 0402WGF0000TCE
- added R11: 0805W8F1004T5E, pepy_sym_lib:[RES_SMD_0805_2012Metric], symbol pepy_sym_lib:[RES_SMD_0805_2012Metric]UNI-ROYAL(Uniroyal Elec) 0805W8F1004T5E
- added R12: RK73H2ATTD3573F, pepy_sym_lib:[RES_SMD_0805_2012Metric], symbol pepy_sym_lib:[RES_SMD_0805_2012Metric]KOA Speer Elec RK73H2ATTD3573F
- added R3: 0805W8F1002T5E, pepy_sym_lib:[RES_SMD_0805_2012Metric], symbol pepy_sym_lib:[RES_SMD_0805_2012Metric]UNI-ROYAL(Uniroyal Elec) 0805W8F1002T5E
- added R4, R5: 0805W8F0000T5E, pepy_sym_lib:[RES_SMD_0805_2012Metric], symbol pepy_sym_lib:[RES_SMD_0805_2012Metric]UNI-ROYAL(Uniroyal Elec) 0805W8F0000T5E
- added RF2, RF3: U.FL-R-SMT-1(80), pepy_sym_lib:[SMD_COAXIAL_CONNECTOR]HRS(Hirose) U.FL-R-SMT-1(80), symbol pepy_sym_lib:[SMD_COAXIAL_CONNECTOR]HRS(Hirose) U.FL-R-SMT-1(80)
- added S1: TS-1088-AR02016, pepy_sym_lib:[TACTILE_SWITCH]XUNPU TS-1088-AR02016, symbol pepy_sym_lib:[TACTILE_SWITCH]XUNPU TS-1088-AR02016
- added U1: AP2114HA-3.3TRG1, pepy_sym_lib:[LDO]Diodes Incorporated AP2114HA-3.3TRG1, symbol pepy_sym_lib:[LDO]Diodes Incorporated AP2114HA-3.3TRG1
- added U3: PMW3360DM-T2QU, pepy_sym_lib:[OPTICAL_NAVIGATION_CHIP]PixArt PMW3360DM-T2QU, symbol pepy_sym_lib:[OPTICAL_NAVIGATION_CHIP]PixArt PMW3360DM-T2QU
- added U4: TPS61220DCKR, pepy_sym_lib:[BOOST_CONV]Texas Instruments TPS61220DCKR, symbol pepy_sym_lib:[BOOST_CONV]Texas Instruments TPS61220DCKR
- added X3: WJ500V-5.08-2P-14-00A, pepy_sym_lib:[1x2_SCREW_TERMINAL_BLOCK]Ningbo Kangnex Elec WJ500V-5.08-2P, symbol pepy_sym_lib:[1x2_SCREW_TERMINAL_BLOCK]Ningbo Kangnex Elec WJ500V-5.08-2P
- C11, C8: value 100pF -> C_Small
- C9: value 4.7u -> C_Small
- J1: renamed from J?; MANUFACTURER (none) -> Tag-Connect; PARTREV (none) -> A; STANDARD (none) -> Manufacturer recommendations
- gave numbers to parts that had none: 15
Connections:
- net BUTTON: now also U2.6 (P0.06); no longer U2.13 (P0.16)
- net GEN1: now also U2.7 (P0.09); no longer U2.14 (P0.18)
- net GND: now also ANT2.1 (GND), C1.1, C15.1, C16.1, C17.1, C18.1, C19.2, C2.1, C20.1, C3.1, R12.1, RF2.2 (GND), RF2.3 (GND), RF3.2 (GND), RF3.3 (GND), S1.1, U1.2 (GND), U1.4 (GND), U3.8 (GND), U4.3 (GND), X3.2; no longer J1.5
- net P0.20: now also Q1.1 (G); no longer R2.1, U2.15 (P0.20)
- net nRESET: now also R4.1
- net at R2.2: now also Q1.3 (D); no longer D2.1 (A)
- net SCK: now reaches U2.10 (P0.12)
- net MOSI: now reaches U2.11 (P0.14)
- net MISO: now reaches U2.12 (P0.15)
- net ANT: now reaches U2.19 (ANT)
- net ANT: now also R10.1
- net nRST_MAN: now reaches U2.8 (P0.10)
- net nRST_MAN: now also R5.1
- net +3.3V renamed VDD_MCU
- net VDD_MCU: now also R3.2, U3.5 (VDDIO); no longer R1.1
- net V_INPUT renamed VDBG
- net VDBG: now also H1.1
- new net: ANT2.2 (SGN), R6.2, R7.2
- new net: L2.1, U4.5 (L)
- new net: C18.2, C19.1, U3.3 (VDDPIX)
- new net: R7.1, RF2.1 (SIG)
- new net: L1.1, R8.1
- new net: C15.2, R6.1, R8.2
- new net: R9.1, RF3.1 (SIG)
- new net: C16.2, L1.2, R10.2, R9.2
- new net: D2.1 (A), Q1.2 (S)
- new net: R11.1, R12.2, U4.2 (FB)
- new net CS: U2.13 (P0.16)
- new net LEFT: C3.2, R3.1, S1.2
- new net MTN_INT: U2.14 (P0.18), U3.9 (MOTION)
- new net VBAT: H3.1
- new net VDD_1.9V: C20.2, R11.2, U3.4 (VDD), U4.4 (VOUT)
- new net VDD_3.3V: C2.2, U1.3 (OUT)
- new net VEXT: H2.1, X3.1
- new net VIN: C17.2, H1.2, H2.2, H3.2, L2.2, R1.1, R2.1, U4.1 (VIN), U4.6 (EN)
- new net VIN_LDO: C1.2, U1.1 (IN)
- new net nRST_PMW: R4.2, R5.2, U3.7 (NRESET)
- no-connect marks 16 -> 14
Other:
- note added: "AUX power"
- note added: "Flags"
- note added: "Main power supply"
- note added: "Power selector"
- note added: "User LED"
- note added: "VINPUT: - On-board power supply (adjustable from external power supply) - 2x AA battery (~3.3V) - Power supply via debug header (adjustable)"
- note removed: "LED"
- note removed: "Power section"
- moved on the sheet: C10, C11, C12, C13, C14, C4, C5, C6, C7, C8, C9, FID1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

Commit message: First draft design
Parts:
- removed C11, C8, C9: C_Small, Capacitor_SMD:C_0805_2012Metric, symbol Device:C_Small
- removed R7: 0402WGF0000TCE, pepy_sym_lib:[RES_SMD_0402_1005Metric], symbol pepy_sym_lib:[RES_SMD_0402_1005Metric]UNI-ROYAL(Uniroyal Elec) 0402WGF0000TCE
- removed U2: NRF52810-QCAA-R, my_lib:[MCU]Nordic Semicon nRF52810-QCAA-R, symbol my_symbol_library:NRF52810-QCAA-R
- removed X1: SC-20S32.768kHz20PPM9pF, my_lib:[Crystal_32_768_kHZ]Seiko SC-20S,32.768kHz,20PPM,9pF, symbol my_symbol_library:SC-20S32.768kHz20PPM9pF
- added C12: CC0805KRX7R9BB104, pepy_sym_lib:[CAP_SMD_0805_2012Metric], symbol pepy_sym_lib:[CAP_SMD_0805_2012Metric]YAGEO CC0805KRX7R9BB104
- added C13: C0805C101K5GACTU, pepy_sym_lib:[CAP_SMD_0805_2012Metric], symbol pepy_sym_lib:[CAP_SMD_0805_2012Metric]KEMET C0805C101K5GACTU
- added C20: C0805C105M4VACTU, pepy_sym_lib:[CAP_SMD_0805_2012Metric], symbol pepy_sym_lib:[CAP_SMD_0805_2012Metric]KEMET C0805C105M4VACTU
- added C6: CL21A475KAQNNNE, pepy_sym_lib:[CAP_SMD_0805_2012Metric], symbol pepy_sym_lib:[CAP_SMD_0805_2012Metric]Samsung Electro-Mechanics CL21A475KAQNNNE
- added R10, R9: 0805W8F1002T5E, pepy_sym_lib:[RES_SMD_0805_2012Metric], symbol pepy_sym_lib:[RES_SMD_0805_2012Metric]UNI-ROYAL(Uniroyal Elec) 0805W8F1002T5E
- added R6: 0402WGF0000TCE, pepy_sym_lib:[RES_SMD_0402_1005Metric], symbol pepy_sym_lib:[RES_SMD_0402_1005Metric]UNI-ROYAL(Uniroyal Elec) 0402WGF0000TCE
- added R8: 0805W8F1000T5E, pepy_sym_lib:[RES_SMD_0805_2012Metric], symbol pepy_sym_lib:[RES_SMD_0805_2012Metric]UNI-ROYAL(Uniroyal Elec) 0805W8F1000T5E
- added S1: TS-1088-AR02016, pepy_sym_lib:[TACTILE_SWITCH]XUNPU TS-1088-AR02016, symbol pepy_sym_lib:[TACTILE_SWITCH]XUNPU TS-1088-AR02016
- added U1: NRF52810-QCAA-R, pepy_sym_lib:[MCU]Nordic Semicon nRF52810-QCAA-R, symbol pepy_sym_lib:[MCU]Nordic Semicon nRF52810-QCAA-R
- added X2: SC-20S32.768kHz20PPM9pF, pepy_sym_lib:[Crystal_32_768_kHZ]Seiko SC-20S,32.768kHz,20PPM,9pF, symbol pepy_sym_lib:[Crystal_32_768_kHZ]Seiko SC-20S,32.768kHz,20PPM,9pF
- R5: renamed from R9; now not fitted
- renumbered ANT2 to ANT1, C16 to C1, C12 to C10, C7 to C11, C19 to C14, C18 to C15, C1 to C16, C2 to C17, C17 to C18, C20 to C19, C15 to C2, C3 to C21, C14 to C3, C13 to C4, C6 to C5, C10 to C7, C4 to C8, C5 to C9, H3 to H2, H2 to H3, R3 to R11, R11 to R12, R4 to R13, R12 to R14, R5 to R15, R10 to R2, R8 to R3, R6 to R4, R2 to R7, RF2 to RF1, RF3 to RF2, S1 to S2, U3 to U2, U1 to U3, X2 to X1
Connections:
- net ANT: now also U1.19 (ANT)
- net GND: now also C8.1, C12.1, C13.1, C20.1, C6.1, S1.1, U1.20 (VSS), U1.29 (VSS), U1.33 (EP); no longer C8.2
- net LEFT: now also C20.2, R10.1, S1.2, U1.5 (P0.05/AIN3); no longer C21.2, R11.1, S2.2
- net MISO: now also U2.12 (MISO), R9.2, U1.12 (P0.15)
- net MOSI: now also U2.11 (MOSI), U1.11 (P0.14)
- net MTN_INT: now also U1.14 (P0.18)
- net SWDCLK: now also U1.17 (SWDCLK)
- net SWDIO: now also U1.18 (SWDIO)
- net VDD_1.9V: now also H5.1, R8.2
- net VDD_3.3V: now also H6.1
- net VDD_MCU: now also H5.2, H6.2, C6.2, R10.2, R9.1, U1.25 (VDD), U1.32 (VDD), U1.9 (VDD)
- net VIN: now also H4.1
- net VIN_LDO: now also H4.2
- net XC1: now also U1.23 (XC1)
- net XC2: now also U1.24 (XC2)
- net nRESET: now also U1.16 (P0.21/nRESET)
- net nRST_MAN: now also U1.8 (P0.10)
- net at ANT1.2 (SGN), R4.2: now also R6.2
- net at RF1.1 (SIG): now also R6.1
- net at C5.2: now also U1.1 (DEC1)
- net at C9.2: now also U1.3 (P0.01/XL2), X2.2
- net at C7.2: now also U1.30 (DEC4)
- net GEN: now reaches J1.5
- net GEN: now also U1.7 (P0.09)
- net SCLK: now reaches U2.10 (SCLK)
- net SCLK: now also U1.10 (P0.12)
- net nCS: now reaches U2.13 (NCS)
- net nCS: now also U1.13 (P0.16)
- net at U2.15 (LED_P): now also R8.1
- net P0.20 renamed LED
- net LED: now also U1.15 (P0.20)
- new net: C12.2, U1.21 (DEC2)
- new net: C8.2, U1.2 (P0.00/XL1), X2.1
- new net: C13.2, U1.22 (DEC3)
- new net RIGHT: C21.2, R11.1, S2.2, U1.6 (P0.06)
- no-connect marks 14 -> 13
Other:
- note added: "Antenna"
- note added: "Left click"
- note added: "Optical sensor"
- note added: "Right click"
- note added: "nRST for PMW sensor"
- note removed: "Button"
- moved on the sheet: ANT1, C1, C10, C11, C14, C15, C2, C21, C3, C4, C5, C7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

Commit message: bump large
Parts:
- removed R9: 0805W8F1002T5E, pepy_sym_lib:[RES_SMD_0805_2012Metric], symbol pepy_sym_lib:[RES_SMD_0805_2012Metric]UNI-ROYAL(Uniroyal Elec) 0805W8F1002T5E
- removed X1: XL7EL89CKI-111YLC-32M, my_lib:[Crystal_32_MHz]YXC XL7EL89CKI-111YLC-32M, symbol my_symbol_library:XL7EL89CKI-111YLC-32M
- added C22, C23: CC0805KRX7R9BB104, pepy_sym_lib:[CAP_SMD_0805_2012Metric], symbol pepy_sym_lib:[CAP_SMD_0805_2012Metric]YAGEO CC0805KRX7R9BB104
- added MH4: ~, pepy_sym_lib:[MOUNTING_HOLE]MountingHole_2.2mm_M2_DIN965_Pad, symbol pepy_sym_lib:[MOUNTING_HOLE]MountingHole_Pad
- added TP1: VBAT, pepy_sym_lib:[TEST_POINT]TestPoint_Pad_2.0x2.0mm, symbol pepy_sym_lib:[TEST_POINT]TestPoint
- added TP2: GND, pepy_sym_lib:[TEST_POINT]TestPoint_Pad_2.0x2.0mm, symbol pepy_sym_lib:[TEST_POINT]TestPoint
- added X1: XL7EL89CKI-111YLC-32M, pepy_sym_lib:[Crystal_32_MHz]YXC XL7EL89CKI-111YLC-32M, symbol pepy_sym_lib:[Crystal_32_MHz]YXC XL7EL89CKI-111YLC-32M
- C3, C4, C8, C9: LCSC Part C1713 -> C3844403; Manufacturer KEMET -> KEMET
Connections:
- net GND: now also C22.1, C23.1, MH4.1, TP2.1, X1.2 (GND), X1.4 (GND)
- net MISO: now also U1.11 (P0.14); no longer U1.12 (P0.15)
- net MOSI: now also U1.12 (P0.15); no longer U1.11 (P0.14)
- net SCLK: now also U1.13 (P0.16); no longer U1.10 (P0.12)
- net VBAT: now also TP1.1
- net VDD_1.9V: now also C23.2
- net VDD_MCU: now also C22.2
- net XC1: now also X1.1
- net XC2: now also X1.3
- net nCS: now also U1.10 (P0.12); no longer U1.13 (P0.16)
- no-connect marks 13 -> 8
Other:
- note added: "Battery"
- company: (none) -> Daniel Hatar
- title: (none) -> Mouse BT HID 

Commit message: Bulk change
Connections:
- net GEN: now also U1.8 (P0.10); no longer U1.7 (P0.09)
- net LED: now also U1.7 (P0.09); no longer U1.15 (P0.20)
- net nRST_MAN: now also U1.15 (P0.20); no longer U1.8 (P0.10)
Changed lines of the file:
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@@
 	)
 	(label "GEN"
-		(at 95.25 48.26 180)
+		(at 95.25 50.8 180)
 		(fields_autoplaced yes)
 		(effects
@@
 	)
 	(label "nRST_MAN"
-		(at 95.25 50.8 180)
+		(at 95.25 68.58 180)
 		(fields_autoplaced yes)
 		(effects
@@
 	)
 	(label "LED"
-		(at 95.25 68.58 180)
+		(at 95.25 48.26 180)
 		(fields_autoplaced yes)
 		(effects
@@
 		)
 	)
+	(netclass_flag ""
+		(length 2.54)
+		(shape dot)
+		(at 280.67 24.13 0)
+		(fields_autoplaced yes)
+		(effects
+			(font
+				(size 1.27 1.27)
+			)
+			(justify left bottom)
+		)
+		(property "Netclass" "Zcontcoplan"
+			(at 281.3685 21.59 0)
+			(effects
+				(font
+					(size 1.27 1.27)
+					(italic yes)
+				)
+				(justify left)
+				(hide yes)
+			)
+		)
+	)
+	(netclass_flag ""
+		(length 2.54)
+		(shape dot)
+		(at 238.76 24.13 0)
+		(fields_autoplaced yes)
+		(effects
+			(font
+				(size 1.27 1.27)
+			)
+			(justify left bottom)
+		)
+		(property "Netclass" "Zcontcoplan"
+			(at 239.4585 21.59 0)
+			(effects
+				(font
+					(size 1.27 1.27)
+					(italic yes)
+				)
+				(justify left)
+			)
+		)
+	)
+	(netclass_flag ""
+		(length 2.54)
+		(shape dot)
+		(at 231.14 39.37 90)
+		(fields_autoplaced yes)
+		(effects
+			(font
+				(size 1.27 1.27)
+			)
+			(justify left bottom)
+		)
+		(property "Netclass" "Zcontcoplan"
+			(at 228.6 38.6715 90)
+			(effects
+				(font
+					(size 1.27 1.27)
+					(italic yes)
+				)
+				(justify left)
+				(hide yes)
+			)
+		)
+	)
+	(netclass_flag ""
+		(length 2.54)
+		(shape dot)
+		(at 299.72 24.13 0)
+		(fields_autoplaced yes)
+		(effects
+			(font
+				(size 1.27 1.27)
+			)
+			(justify left bottom)
+		)
+		(property "Netclass" "Zcontcoplan"
+			(at 300.4185 21.59 0)
+			(effects
+				(font
+					(size 1.27 1.27)
+					(italic yes)
+				)
+				(justify left)
+				(hide yes)
+			)
+		)
+	)
+	(netclass_flag ""
+		(length 2.54)
+		(shape dot)
+		(at 299.72 35.56 90)
+		(fields_autoplaced yes)
+		(effects
+			(font
+				(size 1.27 1.27)
+			)
+			(justify left bottom)
+		)
+		(property "Netclass" "Zcontcoplan"
+			(at 297.18 34.8615 90)
+			(effects
+				(font
+					(size 1.27 1.27)
+					(italic yes)
+				)
+				(justify left)
+				(hide yes)
+			)
+		)
+	)
+	(netclass_flag ""
+		(length 2.54)
+		(shape dot)
+		(at 303.53 24.13 0)
+		(fields_autoplaced yes)
+		(effects
+			(font
+				(size 1.27 1.27)
+			)
+			(justify left bottom)
+		)
+		(property "Netclass" "Zcontcoplan"
+			(at 304.2285 21.59 0)
+			(effects
+				(font
+					(size 1.27 1.27)
+					(italic yes)
+				)
+				(justify left)
+				(hide yes)
+			)
+		)
+	)
+	(netclass_flag ""
+		(length 2.54)
+		(shape dot)
+		(at 269.24 24.13 0)
+		(fields_autoplaced yes)
+		(effects
+			(font
+				(size 1.27 1.27)
+			)
+			(justify left bottom)
+		)
+		(property "Netclass" "Zcontcoplan"
+			(at 269.9385 21.59 0)
+			(effects
+				(font
+					(size 1.27 1.27)
+					(italic yes)
+				)
+				(justify left)
+				(hide yes)
+			)
+		)
+	)

Commit message: test_phase
Parts:
- added TP3: Vtref, pepy_sym_lib:[TEST_POINT]TestPoint_Pad_D1.0mm, symbol pepy_sym_lib:[TEST_POINT]TestPoint
- added TP4: LED, pepy_sym_lib:[TEST_POINT]TestPoint_Pad_D1.0mm, symbol pepy_sym_lib:[TEST_POINT]TestPoint
- added TP5: LEFT, pepy_sym_lib:[TEST_POINT]TestPoint_Pad_D1.0mm, symbol pepy_sym_lib:[TEST_POINT]TestPoint
- added TP6: RIGHT, pepy_sym_lib:[TEST_POINT]TestPoint_Pad_D1.0mm, symbol pepy_sym_lib:[TEST_POINT]TestPoint
- added TP7: nRESET, pepy_sym_lib:[TEST_POINT]TestPoint_Pad_D1.0mm, symbol pepy_sym_lib:[TEST_POINT]TestPoint
Connections:
- net LED: now also TP4.1
- net LEFT: now also TP5.1
- net RIGHT: now also TP6.1
- net VDD_MCU: now also TP3.1
- net nRST_PMW: now also TP7.1
